Commit message: added 2wheel urdf

File: urdf/gazebo.xacro (robot description, xacro)
@@ -1,4 +1,4 @@
 <?xml version="1.0"?>
-<robot xmlns:xacro="http://www.ros.org/wiki/xacro" name="bcr_bot">
+<robot xmlns:xacro="http://www.ros.org/wiki/xacro" name="diffbot">
     <!-- ........................... SENSOR PLUGIN ................................... -->
     <gazebo>
@@ -23,9 +23,13 @@
             <child_frame_id>base_footprint</child_frame_id>
         </plugin> -->
-        <plugin filename="diffdriveplugin" name="wheel_rpm_plugin::WheelRPMPlugin">
-            <left_joint_name>front_left_wheel_joint</left_joint_name>
-            <right_joint_name>front_right_wheel_joint</right_joint_name>
+        <plugin filename="libCustomDiffDrive.so" name="custom::CustomDiffDrive">
+            <!-- <left_wheel_joint>front_left_wheel_joint</left_wheel_joint>
+            <right_wheel_joint>front_right_wheel_joint</right_wheel_joint> -->
+            <left_wheel_joint>left_wheel_joint</left_wheel_joint>
+            <right_wheel_joint>right_wheel_joint</right_wheel_joint>
             <left_rpm_topic>/left_wheel_rpm</left_rpm_topic>
             <right_rpm_topic>/right_wheel_rpm</right_rpm_topic>
+            <wheel_radius>0.2</wheel_radius>
+            <wheel_base>1.1</wheel_base>
         </plugin>
     </gazebo>

File: urdf/materials.xacro (robot description, xacro)
@@ -40,3 +40,6 @@
         <color rgba="0.1 0.1 0.1 1"/>
     </material>
+    <material name ='wooden'>
+        <color rgba='0.76 0.60 0.024 1'/>
+    </material>
 </robot>

File: urdf/robot_sim.xacro (robot description, xacro)
@@ -77,5 +77,5 @@
         </inertial>
     </link>
-    <joint name="rear_left_wheel_joint" type="continuous">
+    <joint name="rear_left_wheel_joint" type="continuous"> <!--continuous-->
         <parent link="chassis_link"/>
         <child link="rear_left_wheel"/>
@@ -126,5 +126,5 @@
         </inertial>
     </link>
-    <joint name="rear_right_wheel_joint" type="continuous">
+    <joint name="rear_right_wheel_joint" type="continuous"> <!--continuous-->
         <parent link="chassis_link"/>
         <child link="rear_right_wheel"/>

Commit message: new sensors plugins added

File: urdf/gazebo.xacro (robot description, xacro)
@@ -64,7 +64,12 @@
                         <max_angle>3.14</max_angle>
                     </horizontal>
+                    <vertical>
+                        <samples>32</samples>
+                        <min_angle>-0.5353</min_angle>
+                        <max_angle>0.1862</max_angle>
+                    </vertical>
                 </scan>
                 <range>
-                    <min>0.1</min>
+                    <min>1.1</min>
                     <max>10.0</max>
                     <resolution>0.01</resolution>
@@ -81,13 +86,12 @@
     </gazebo>
     <!-- ........................... CAMERA config ................................... -->
-    <!-- <xacro:if value="$(arg camera_enabled)"> -->
-    <!-- <gazebo reference="kinect_camera">
-        <sensor type="depth_camera" name="kinect_camera">
+    <!-- <gazebo reference="camera">
+        <sensor type="camera" name="camera">
             <update_rate>30.0</update_rate>
-            <topic>kinect_camera</topic>
-            <gz_frame_id>kinect_camera</gz_frame_id>
+            <topic>camera/image</topic>
+            <gz_frame_id>camera</gz_frame_id>
             <camera>
-                <camera_info_topic>kinect_camera/camera_info</camera_info_topic>
-                <horizontal_fov>${radians(camera_horizontal_fov)}</horizontal_fov>
+                <camera_info_topic>camera/camera_info</camera_info_topic>
+                <horizontal_fov>1.047</horizontal_fov>
                 <image>
                     <width>640</width>
@@ -102,6 +106,27 @@
         </sensor>
     </gazebo> -->
+      <gazebo reference="camera">
+        <sensor name="rgbd_camera" type="rgbd_camera">
+        <camera>
+            <horizontal_fov>1.25</horizontal_fov>
+            <image>
+                <width>640</width>
+                <height>480</height>
+            </image>
+            <clip>
+                <near>0.1</near>
+                <far>15</far>
+            </clip>
+            <optical_frame_id>camera_optical</optical_frame_id>
+        </camera>
+        <always_on>1</always_on>
+        <update_rate>20</update_rate>
+        <visualize>true</visualize>
+        <topic>camera</topic>
+        <gz_frame_id>camera</gz_frame_id>
+        </sensor>
+    </gazebo>
     <!-- ........................... IMU config ................................... -->
-    <!-- <gazebo reference="imu_frame">
+    <gazebo reference="imu_frame">
         <sensor name="imu_sensor" type="imu">
             <always_on>1</always_on>
@@ -111,5 +136,5 @@
             <topic>imu</topic>
         </sensor>
-    </gazebo> -->
+    </gazebo>
     <!-- ........................... Stereo camera ................................... -->
     <!-- <gazebo reference="stereo_camera">

File: urdf/robot_sim.xacro (robot description, xacro)
@@ -181,3 +181,33 @@
         <origin xyz="0.0 0.0 0.16" rpy="0.0 0.0 0.0"/>
     </joint>
+    <link name="camera">
+        <collision>
+            <origin xyz="0 0 0" rpy="0 0 0" />
+            <geometry>
+                <box size="0.07 0.3 0.09"/>
+            </geometry>
+        </collision>
+        <visual>
+            <origin xyz="0 0 0" rpy="0 0 0" />
+            <geometry>
+                <mesh filename="file://$(find diffbot)/meshes/camera/d415.dae"/>
+            </geometry>
+            <material name="black"/>
+        </visual>
+        <inertial>
+            <mass value="0.01"/>
+            <xacro:box_inertia m="0.01" x="0.07" y="0.3" z = "0.09"/>
+        </inertial>
+    </link>
+    <joint name="camera_joint" type="fixed">
+        <origin rpy="0 0 0" xyz="0.78 0 0.0428"/>
+        <parent link="base_link"/>
+        <child link="camera"/>
+    </joint>
+    <link name="camera_optical"/>
+    <joint name="camera_optical_joint" type="fixed">
+        <origin xyz="0 0 0" rpy="0 0 0"/>
+        <parent link="camera"/>
+        <child link="camera_optical"/>
+    </joint>
 </robot>
